File: hardware/DummyLoadV2/DummyLoadV2_Digital.kicad_sch (KiCad schematic)
At the start: 18 parts, among them J1 Conn_01x05_Pin, J2 Fan, Q3 2N7000, Q4 PMOS, SW1 Enable_SW, SW3 Range_SW, U1 Nano

Commit message: Updated schematic
Parts:
- removed J1: Conn_01x05_Pin, symbol Connector:Conn_01x05_Pin
- removed J2: Fan, symbol Connector:Conn_01x04_Pin
- added J3: Display, symbol Connector_Generic:Conn_01x05
- added J4: Digital, symbol Connector_Generic:Conn_02x04_Top_Bottom
- added J7: Fan, symbol Connector_Generic:Conn_01x04
- Q4: value PMOS -> TP2104
- R8: value 100k -> 10k
Connections:
- net Fan_PWM: now also J7.4 (Pin_4)
- net Fan_Tach: now also J7.3 (Pin_3)
- net GND: now also J3.5 (Pin_5), J7.1 (Pin_1)
- net Output_Relay: now also U1.20 (A1), J4.7 (Pin_7); no longer U1.19 (A0)
- net Range_Relay: now also U1.21 (A2), J4.8 (Pin_8); no longer U1.20 (A1)
- net VDD: now also J3.4 (Pin_4), J4.6 (Pin_6)
- net at NTC.1, R9.2: now also U1.25 (A6); no longer U1.26 (A7)
- net at Q4.3 (S): now also J7.2 (Pin_2)
- net MOSI: now reaches U1.14 (D11)
- net MOSI: now also J3.1 (Pin_1), J4.2 (Pin_2)
- net SCK: now reaches U1.16 (D13)
- net SCK: now also J3.2 (Pin_2), J4.3 (Pin_3)
- net Display_CS: now reaches U1.13 (D10)
- net Display_CS: now also J3.3 (Pin_3)
- net MISO: now reaches U1.15 (D12)
- net MISO: now also J4.1 (Pin_1)
- net ADC_CS: now reaches U1.22 (A3)
- net ADC_CS: now also J4.5 (Pin_5)
- net SCL: no longer names the net of U1.24 (A5)
- net SDA: no longer names the net of U1.23 (A4)
- new net DAC_CS: J4.4 (Pin_4), U1.19 (A0)
- no-connect marks 10 -> 9
Other:
- moved on the sheet: C4, C5, C6, C7, C8, C9, ENC1, NTC, Q3, Q4, R7, R8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

Commit message: Updated schematic
Other:
- moved on the sheet: C4, C5, C6, C7, C8, C9, ENC1, J3, J4, J7, NTC, Q3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
